File: EAGLE/MSSRP-Sensor/MSSRP-TC_IF.sch (EAGLE design)
At the start: 0 parts

Commit message: Update 3
Added Main Board Files
Parts:
- added C1, C4: 0.1uF, SparkFun-Capacitors:0.1UF-25V-5%(0603)
- added C2, C5: 1.0uF, SparkFun-Capacitors:1.0UF-16V-10%(0603)
- added C3, C6: 10nF, SparkFun-Capacitors:10NF/10000PF-50V-10%(0603)
- added R1, R2, R3, R4, R5, R6: 0, SparkFun-Resistors:0OHM1/10W5%(0603)
- added U$1, U$2: MAX6675, SparkFun-AnalogIC:MAX6675
Connections:
- new net 3.3V: C1.2, C2.2, C4.2, C5.2, U$1.VDD, U$2.VDD
- new net AIN0+: C3.1, U$1.T+
- new net AIN0-: C3.2, U$1.T-
- new net AIN1+: C6.1, U$2.T+
- new net AIN1-: C6.2, U$2.T-
- new net CS0: R2.1
- new net CS1: R5.1
- new net GND: C1.1, C2.1, C4.1, C5.1, U$1.VSS, U$2.VSS
- new net MISO: R3.1, R6.1
- new net N$1: R3.2, U$1.MISO
- new net N$10: R5.2, U$2.CS
- new net N$11: R4.2, U$2.SCK
- new net N$2: R2.2, U$1.CS
- new net N$3: R1.2, U$1.SCK
- new net N$9: R6.2, U$2.MISO
- new net SCK: R1.1, R4.1
