File: EAGLE/MSSRP-Sensor/MSSRP-Temperature_System_beta.sch (EAGLE design)
At the start: 225 parts, among them J1 POWER_JACKPTH, J10 BNCPTH, J11 BNCPTH, J2 USBSMD, J4 TE-2-TERMBLOCK, J5 TE-2-TERMBLOCK, J6 TE-2-TERMBLOCK, J7 TE-2-TERMBLOCK, J8 BNCPTH, J9 BNCPTH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

Commit message: Layout start
Some schematic changes, eliminating several 0-ohm “oops” resistors.
General layout OK, initial routing started.
Parts:
- removed C31: 0.1uF, SparkFun-Capacitors:0.1UF-25V-5%(0603)
- removed R125, R126, R127, R129, R131, R132, R53, R54, R58, R59, R60, R61, R62, R63, R64, R65, R66, R67, R68, R69, R70, R71, R72, R74: 0, SparkFun-Resistors:0OHM1/10W5%(0603)
- removed TP1, TP2: TPPAD1-13, testpad:TPPAD1-13
- C15: value 10uF -> 4.7uF; device SparkFun-Capacitors:10UF-16V-10%(TANT) -> SparkFun-Capacitors:4.7UF-6.3V-10%(0603)0603
Connections:
- removed net AFE_D0: R63.2
- removed net AFE_D1: R62.2
- removed net AFE_D2: R61.2
- removed net AFE_D3: R60.2
- removed net N$127: J2.D-, TP2.TP
- removed net N$128: J2.D+, TP1.TP
- removed net N$129: J8.OUT, R126.2
- removed net N$130: J9.OUT, R125.2
- removed net N$131: J7.1, R127.2
- removed net N$132: J7.2, R128.2
- removed net N$133: J6.1, R129.2
- removed net N$134: J6.2, R130.2
- removed net N$49: R53.1, U4.!SYNC!/!PWDN
- removed net N$50: R54.1, U4.!RESET
- removed net N$54: R58.1, U4.!DRDY
- removed net N$55: R59.1, U4.!CS
- removed net N$56: R60.1, U4.D3
- removed net N$57: R61.1, U4.D2
- removed net N$58: R62.1, U4.D1
- removed net N$59: R63.1, U4.D0/CLKOUT
- removed net N$60: R64.2, U4.AIN0
- removed net N$61: R65.2, U4.AIN1
- removed net N$62: R66.2, U4.AIN2
- removed net N$63: R67.2, U4.AIN3
- removed net N$64: R68.2, U4.AIN4
- removed net N$65: R69.2, U4.AIN5
- removed net N$66: R70.2, U4.AIN6
- removed net N$67: R71.2, U4.AIN7
- removed net N$68: R72.2, U4.AINCOM
- removed net N$70: R74.2, U4.VREFN
- removed net N$84: R23.2
- net 5V: now also C15.1; no longer C15.+
- net AFE_!DRDY: now also U4.!DRDY; no longer R58.2
- net AFE_!PWDN: now also U4.!SYNC!/!PWDN; no longer R53.2
- net AFE_!RESET: now also R23.2, U4.!RESET; no longer R54.2
- net AFE_AIN0: now also J6.1, J8.OUT, U4.AIN0; no longer R126.1, R129.1, R64.1
- net AFE_AIN1: now also J6.2, J8.GND, R130.2, U4.AIN1; no longer R130.1, R131.1, R65.1
- net AFE_AIN2: now also J7.1, J9.OUT, U4.AIN2; no longer R125.1, R127.1, R66.1
- net AFE_AIN3: now also J7.2, J9.GND, R128.2, U4.AIN3; no longer R128.1, R132.1, R67.1
- net CS_AFE: now also U4.!CS; no longer R59.2
- net GND: now also C15.2, R128.1, R130.1, U4.AINCOM, U4.VREFN; no longer C15.-, C31.1, J8.GND, J9.GND, R131.2, R132.2, R68.1, R69.1, R70.1, R71.1, R72.1, R74.1
- net VUSB: no longer C31.2, J2.VBUS, U1.P$39
Other:
- moved on the sheet: R128, R130, R73

Commit message: Updated routing
Schematic and routing edits. Core power routing done.
Parts:
- removed C36: 10uF, SparkFun-Capacitors:10UF-16V-10%(TANT)
- removed LED1, LED2: (no value), SparkFun-LED:LED0603
- removed R121, R122, R123, R124, R29, R30, R31, R32, R80, R83, R87, R89: 0, SparkFun-Resistors:0OHM1/10W5%(0603)
- removed R96, R97: 470, SparkFun-Resistors:470OHM1/10W1%(0603)
- removed S1: SWITCH-MOMENTARY-2-SMD-1101NE, SparkFun-Electromechanical:SWITCH-MOMENTARY-2-SMD-1101NE
- added C31: 4.7uF, SparkFun-Capacitors:4.7UF-6.3V-10%(0603)0603
- C8: value 10uF -> 4.7uF; device SparkFun-Capacitors:10UF-16V-10%(TANT) -> SparkFun-Capacitors:4.7UF-6.3V-10%(0603)0603
Connections:
- net N$108 renamed VBATT
- net N$96 renamed VLDO
- removed net BATT_!CHG: R17.1
- removed net BICOLOR_LED0: R27.2
- removed net BICOLOR_LED1: R28.2
- removed net CS_BT: R30.1, R5.1
- removed net N$122: R121.2, U9.!LDAC
- removed net N$123: R122.1, U9.!CLR
- removed net N$125: R123.1, U9.VOUTB
- removed net N$126: R124.1, U9.VOUTA
- removed net N$29: R29.2, U2.SPICLK
- removed net N$31: R31.2, U2.SPIMISO
- removed net N$32: R32.2, U2.SPIMOSI
- removed net N$38: C3.1, R38.2, S1.1, U2.PIO4
- removed net N$76: R76.1, R80.1, U3.SQW
- removed net N$79: R79.1, R83.2, U3.!INTA
- removed net N$80: R87.2, U$1.CS
- removed net N$85: R89.2, U$1.CARD_DETECT
- removed net N$94: LED1.A, R96.1
- removed net N$95: LED2.A, R97.1
- removed net SQW: R20.2
- removed net STATUS_CONN: R96.2
- removed net STATUS_PWR: R26.2, R97.2
- removed net SW1: C29.1, R100.1, R24.2, S2.2
- new net BT_!RESET: C3.1, R38.2, R5.1, U2.PIO4
- new net LED0: R27.2, R98.2
- new net LED1: R28.2, R99.2
- net 3.3V: no longer S1.2
- net CS_SD: now also U$1.CS; no longer R87.1
- net DAC0: now also U9.VOUTA; no longer R124.2
- net DAC1: now also U9.VOUTB; no longer R123.2
- net DAC_!CLR: now also R26.2, U9.!CLR; no longer R122.2
- net DAC_!LDAC: now also R17.1, U9.!LDAC; no longer R121.1
- net GND: now also C31.1, C8.1; no longer C36.-, C8.-, LED1.C, LED2.C
- net MICRO_!RESET: now also C29.1, R100.1, S2.2
- net MISO: no longer R31.1
- net MOSI: no longer R32.1
- net N$30: now also R24.2; no longer R30.2, U2.SPICSB
- net N$5: no longer R98.2
- net N$6: no longer R99.2
- net RTC_!INTA: now also R79.1, U3.!INTA; no longer R83.1
- net RTC_SQW: now also R20.2, R76.1, U3.SQW; no longer R80.2
- net SCK: no longer R29.1
- net SD_CD: now also U$1.CARD_DETECT; no longer R89.1
- net VIN: now also C31.2; no longer C36.+
- net VSYS: now also C8.2; no longer C8.+
- net VUSB: now also U1.P$39
