File: EAGLE/MSSRP-Sensor/MSSRP-Temperature_System_beta_2layer.brd (EAGLE design)
At the start: 100 x 100 mm, 181 parts, among them J1 POWER_JACKPTH, J10 BNCPTH, J11 BNCPTH, J2 USBSMD, J4 TE-2-TERMBLOCK, J5 TE-2-TERMBLOCK, J6 TE-2-TERMBLOCK, J7 TE-2-TERMBLOCK, J8 BNC_CUSTOM, J9 BNC_CUSTOM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

Commit message: Minor changes
Parts:
- Y1: value (none) -> 7.68 MHz
- Y2: value (none) -> 32.768 kHz
Changed lines of the file:
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@@
 <attribute name="VALUE" x="83.693" y="78.994" size="0.4064" layer="27" font="vector" rot="R90"/>
 </element>
-<element name="Y1" library="microbuilder" package="HC49UP" value="" x="64.77" y="69.85"/>
+<element name="Y1" library="microbuilder" package="HC49UP" value="7.68 MHz" x="64.77" y="69.85"/>
 <element name="C19" library="SparkFun-Capacitors" package="0603-CAP" value="18pF" x="67.945" y="66.04" rot="R180">
 <attribute name="PROD_ID" value="CAP-08267" x="-43.815" y="160.02" size="1.778" layer="27" rot="R180" display="off"/>
@@
 </element>
 <element name="U3" library="MSSRP-Lib" package="SOIC8" value="DS1337S+T&amp;R" x="46.99" y="42.545" rot="R180"/>
-<element name="Y2" library="SparkFun-FreqCtrl" package="HC49UP" value="" x="55.245" y="45.72" rot="R270"/>
+<element name="Y2" library="SparkFun-FreqCtrl" package="HC49UP" value="32.768 kHz" x="55.245" y="45.72" rot="R270"/>
 <element name="C21" library="SparkFun-Capacitors" package="0603-CAP" value="0.1uF" x="50.8" y="42.545" rot="R270">
 <attribute name="PROD_ID" value="CAP-08604" x="-46.99" y="23.495" size="1.778" layer="27" rot="R270" display="off"/>
